File: ArduinoToSerial/shields/RJ12_senzor/RJ12_senzor.sch (EAGLE design)
At the start: 2 parts

Commit message: added THT + SMD resistor
Connections:
- net N$1 renamed GND
Changed lines of the file:
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@@
 </busses>
 <nets>
-<net name="N$1" class="0">
+<net name="GND" class="0">
 <segment>
 <pinref part="U$1" gate="G$1" pin="1"/>
